File: esp8266_programmer_tht/esp32_programmer.kicad_sch (KiCad schematic)
At the start: 41 parts, among them P1 USB_C_Plug_USB2.0, Q1 S8050, Q2 S8050, SW1 SW_Push, SW2 SW_Push, U1 CH340C, U2 ESP-12E

Commit message: D+ D- fixing
Connections:
- net at P1.A6 (D+): now also U1.5 (UD+); no longer U1.6 (UD-)
- net at P1.A7 (D-): now also U1.6 (UD-); no longer U1.5 (UD+)
Changed lines of the file:
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@@
+    (stroke (width 0) (type default))
+  )
+  (wire (pts (xy 49.53 48.26) (xy 81.534 48.26))
     (stroke (width 0) (type default))
   )
@@
     (stroke (width 0) (type default))
   )
-  (wire (pts (xy 49.53 48.26) (xy 73.66 48.26))
-    (stroke (width 0) (type default))
-  )
   (wire (pts (xy 96.52 38.1) (xy 96.52 35.56))
     (stroke (width 0) (type default))
@@
     (stroke (width 0) (type default))
   )
+  (wire (pts (xy 81.534 48.26) (xy 84.074 50.8))
+    (stroke (width 0) (type default))
+  )
   (wire (pts (xy 99.06 72.39) (xy 34.29 72.39))
     (stroke (width 0) (type default))
@@
     (stroke (width 0) (type default))
   )
+  (wire (pts (xy 70.104 43.18) (xy 80.264 53.34))
+    (stroke (width 0) (type default))
+  )
   (wire (pts (xy 96.52 35.56) (xy 88.9 35.56))
     (stroke (width 0) (type default))
@@
     (stroke (width 0) (type default))
   )
+  (wire (pts (xy 84.074 50.8) (xy 88.9 50.8))
+    (stroke (width 0) (type default))
+  )
   (wire (pts (xy 33.528 142.24) (xy 33.528 147.066))
     (stroke (width 0) (type default))
@@
     (stroke (width 0) (type default))
   )
-  (wire (pts (xy 49.53 43.18) (xy 76.2 43.18))
+  (wire (pts (xy 49.53 43.18) (xy 70.104 43.18))
     (stroke (width 0) (type default))
   )
@@
     (stroke (width 0) (type default))
   )
-  (wire (pts (xy 76.2 43.18) (xy 76.2 50.8))
-    (stroke (width 0) (type default))
-  )
   (wire (pts (xy 87.63 154.432) (xy 87.63 157.734))
     (stroke (width 0) (type default))
   )
+  (wire (pts (xy 80.264 53.34) (xy 88.9 53.34))
+    (stroke (width 0) (type default))
+  )
   (wire (pts (xy 127 142.24) (xy 138.43 142.24))
     (stroke (width 0) (type default))
@@
     (stroke (width 0) (type default))
   )
-  (wire (pts (xy 73.66 48.26) (xy 73.66 53.34))
-    (stroke (width 0) (type default))
-  )
   (wire (pts (xy 60.96 24.13) (xy 60.96 30.48))
     (stroke (width 0) (type default))
@@
     (stroke (width 0) (type default))
   )
-  (wire (pts (xy 73.66 53.34) (xy 88.9 53.34))
-    (stroke (width 0) (type default))
-  )
   (wire (pts (xy 33.528 134.62) (xy 33.528 133.604))
     (stroke (width 0) (type default))
@@
     (stroke (width 0) (type default))
   )
-  (wire (pts (xy 76.2 50.8) (xy 88.9 50.8))
-    (stroke (width 0) (type default))
-  )
